File: vfd-ps.sch (KiCad schematic (older format))
At the start: 0 parts

Commit message: Draw first schematic
Parts:
- added C?: 100u 16V, symbol Device:CP
- added C?: 150p, symbol Device:C
- added C?: 4.7n, symbol Device:C
- added C?: 220u 35V, symbol Device:CP
- added C?: 10u 16V, symbol Device:C
- added C?: 10n, symbol Device:C
- added C?: 1u, symbol Device:C
- added C? (x2): 22u, symbol Device:CP
- added D?: 40V 3A, symbol Device:D_Schottky
- added D?: 4.7V, symbol Device:D_Zener
- added J? (x3): Conn_01x02, symbol Connector_Generic:Conn_01x02
- added L?: 33u 3A, symbol Device:L_Core_Iron
- added R?: 0.1, symbol Device:R
- added R?: 120k, symbol Device:R
- added R?: 6.2k, symbol Device:R
- added R? (x3): 100, symbol Device:R
- added R?: 2.2k, symbol Device:R
- added R? (x3): 10k, symbol Device:R
- added RV?: 4.7k, symbol Device:R_POT_TRIM
- added RV? (x2): 50, symbol Device:R_POT_TRIM
- added U?: NCP3163PWG, esynr3z_SO:SOIC-16W-1EP_7.5x10.3mm_P1.27mm_ThermalVias, symbol esynr3z_RegulatorSwitching:NCP3163PWG
- added U?: LM4871, esynr3z_SO:VSSOP-8_3.0x3.0mm_P0.65mm, symbol esynr3z_AmplifierAudio:LM4871
Connections:
- net labels added: +5V, GND, VEE, VF1, VF2
- wire segments 0 -> 107
Other:
- note added: "2W @ 5V in"
- note added: "[-15V;-30V] 0.25A @ 5V in"
- note removed: "+5V"
- note removed: "Inverting switching regulator"
- note removed: "Self oscillating filament driver"
- note removed: "To VFD and anode/grid driver"
- note removed: "VEE"
- note removed: "VF1"
- note removed: "VF2"

Commit message: Replace NCP3163 converter with TPS54360
Parts:
- removed C?: 100u 16V, symbol Device:CP
- removed C?: 150p, symbol Device:C
- removed C?: 220u 35V, symbol Device:CP
- removed R?: 0.1, symbol Device:R
- removed R?: 120k, symbol Device:R
- removed R?: 6.2k, symbol Device:R
- removed U?: NCP3163PWG, esynr3z_SO:SOIC-16W-1EP_7.5x10.3mm_P1.27mm_ThermalVias, symbol esynr3z_RegulatorSwitching:NCP3163PWG
- added C1: 22u, symbol Device:C
- added C3: 1u, symbol Device:C
- added C4: 100n, symbol Device:C
- added C5, C6: 4.7u, symbol Device:C
- added C7: 150n, symbol Device:C
- added C8: 1n, symbol Device:C
- added R2: 18k, symbol Device:R
- added R3: dnp, symbol Device:R
- added R4: 100k, symbol Device:R
- added R5: 6.8k, symbol Device:R
- added R6: 1k, symbol Device:R
- added U1: TPS54360DDA, esynr3z_SO:TI_SO-PowerPAD-8_ThermalVias, symbol esynr3z_RegulatorSwitching:TPS54360DDA
- C10: renamed from C?; value 10u 16V -> 22u
- C2: renamed from C?; value 4.7n -> 22u
- L1: renamed from L?; value 33u 3A -> 47u 3A
- R1: renamed from R?; value 100 -> dnp
- RV1: renamed from RV?; value 4.7k -> 20k
- gave numbers to parts that had none: 18
Connections:
- wire segments 107 -> 134

Commit message: Schematic update: footprints, nominals, testpoints, etc
Parts:
- removed D1: 40V 3A, symbol Device:D_Schottky
- removed D2: 4.7V, symbol Device:D_Zener
- added C1: 22u, esynr3z_Capacitor:C_1210, symbol Device:C
- added C8: 4.7u, esynr3z_Capacitor:C_1210, symbol Device:C
- added D1: MBRA340, esynr3z_Diode:SMA, symbol esynr3z_DiodeSchottky:MBRA340
- added D2: BZX84C4V7, esynr3z_SOT:SOT-23, symbol esynr3z_DiodeZener:BZX84C4V7
- added JP1: SolderJumper_2_Bridged, esynr3z_Jumper:SolderJumper-2_P1.3mm_Bridged2Bar_RoundedPad1.0x1.5mm, symbol esynr3z_Misc:SolderJumper_2_Bridged
- added TP1, TP2, TP3: TestPoint, esynr3z_TestPoint:TestPoint_THTPad_D1.5mm_Drill0.7mm, symbol esynr3z_Misc:TestPoint
- C10: renamed from C8; value 1n -> 1.8n; footprint (none) -> esynr3z_Capacitor:C_0805
- C11: renamed from C9; footprint (none) -> esynr3z_Capacitor:CP_Elec_6.3x7.7; Rating (none) -> 50V
- C12: renamed from C10; footprint (none) -> esynr3z_Capacitor:C_1210; Rating (none) -> 16V X5R
- C13: renamed from C11; footprint (none) -> esynr3z_Capacitor:CP_Elec_6.3x7.7; Rating (none) -> 50V
- C14: renamed from C12; footprint (none) -> esynr3z_Capacitor:C_0805
- C15: renamed from C13; footprint (none) -> esynr3z_Capacitor:C_1206
- C2: renamed from C1; footprint (none) -> esynr3z_Capacitor:C_1210; Rating (none) -> 16V X5R
- C3: renamed from C2; footprint (none) -> esynr3z_Capacitor:C_1210; Rating (none) -> 16V X5R
- C4: renamed from C3; footprint (none) -> esynr3z_Capacitor:C_1206; Rating (none) -> 50V X7R
- C5: renamed from C4; footprint (none) -> esynr3z_Capacitor:C_0805
- C6: renamed from C5; footprint (none) -> esynr3z_Capacitor:C_1210; Rating (none) -> 50V X7R
- C7: renamed from C6; footprint (none) -> esynr3z_Capacitor:C_1210; Rating (none) -> 50V X7R
- C9: renamed from C7; value 150n -> 220n; footprint (none) -> esynr3z_Capacitor:C_0805
- J1: renamed from J2; footprint (none) -> esynr3z_Connector:PinHeader_1x02_P2.54mm_Vertical
- J2: renamed from J1; footprint (none) -> esynr3z_Connector:PinHeader_1x02_P2.54mm_Vertical
- J3: footprint (none) -> esynr3z_Connector:PinHeader_1x02_P2.54mm_Vertical
- L1: value 47u 3A -> 33u; footprint (none) -> esynr3z_Inductor:Sumida_CDRH127
- R1, R3: value dnp -> dnf; footprint (none) -> esynr3z_Resistor:R_0805
- R10, R11, R12, R2, R5, R6, R7, R8, R9: footprint (none) -> esynr3z_Resistor:R_0805
- R4: value 100k -> 220k; footprint (none) -> esynr3z_Resistor:R_0805
- RV1, RV2, RV3: footprint (none) -> esynr3z_Potentiometer:Bourns_3362P
Connections:
- wire segments 134 -> 147

Commit message: Minor tweaks in schematic
Parts:
- R2: value 18k -> 16k
Other:
- note added: "Filament driver"
- note added: "Negative supply"

Commit message: Replace connectors, add testpoints, pcb rotate and align
Parts:
- removed J1, J2, J3: Conn_01x02, esynr3z_Connector:PinHeader_1x02_P2.54mm_Vertical, symbol Connector_Generic:Conn_01x02
- added J1, J2, J3: Conn_01x04, esynr3z_Connector:PinHeader_1x04_P2.54mm_Vertical, symbol Connector_Generic:Conn_01x04
- added TP4, TP5: TestPoint, esynr3z_TestPoint:TestPoint_THTPad_D1.5mm_Drill0.7mm, symbol esynr3z_Misc:TestPoint
Connections:
- wire segments 147 -> 163
Changed lines of the file:
@@
 Text GLabel 7000 5000 2    50   Input ~ 0
 VF2
-$Comp
-L Connector_Generic:Conn_01x02 J1
-U 1 1 5B8EFC5A
-P 7700 4100
-F 0 "J1" H 7620 3775 50  0000 C CNN
-F 1 "Conn_01x02" H 7620 3866 50  0000 C CNN
-F 2 "esynr3z_Connector:PinHeader_1x02_P2.54mm_Vertical" H 7700 4100 50  0001 C CNN
-F 3 "~" H 7700 4100 50  0001 C CNN
-	1    7700 4100
-	-1   0    0    1
-$EndComp
-$Comp
-L Connector_Generic:Conn_01x02 J2
-U 1 1 5B8EFEED
-P 7700 4800
-F 0 "J2" H 7620 4475 50  0000 C CNN
-F 1 "Conn_01x02" H 7620 4566 50  0000 C CNN
-F 2 "esynr3z_Connector:PinHeader_1x02_P2.54mm_Vertical" H 7700 4800 50  0001 C CNN
-F 3 "~" H 7700 4800 50  0001 C CNN
-	1    7700 4800
-	-1   0    0    1
-$EndComp
-$Comp
-L Connector_Generic:Conn_01x02 J3
-U 1 1 5B8F1F2E
-P 7700 5400
-F 0 "J3" H 7620 5075 50  0000 C CNN
-F 1 "Conn_01x02" H 7620 5166 50  0000 C CNN
-F 2 "esynr3z_Connector:PinHeader_1x02_P2.54mm_Vertical" H 7700 5400 50  0001 C CNN
-F 3 "~" H 7700 5400 50  0001 C CNN
-	1    7700 5400
-	-1   0    0    1
-$EndComp
-$Comp
-L power:+5V #PWR05
-U 1 1 5B8F438D
-P 8100 3950
-F 0 "#PWR05" H 8100 3800 50  0001 C CNN
-F 1 "+5V" H 8115 4123 50  0000 C CNN
-F 2 "" H 8100 3950 50  0001 C CNN
-F 3 "" H 8100 3950 50  0001 C CNN
-	1    8100 3950
-	1    0    0    -1
-$EndComp
-$Comp
-L power:GND #PWR06
-U 1 1 5B8F64F3
-P 8100 4150
-F 0 "#PWR06" H 8100 3900 50  0001 C CNN
-F 1 "GND" H 8105 3977 50  0000 C CNN
-F 2 "" H 8100 4150 50  0001 C CNN
-F 3 "" H 8100 4150 50  0001 C CNN
-	1    8100 4150
-	1    0    0    -1
-$EndComp
-$Comp
-L power:GND #PWR08
-U 1 1 5B8F84EC
-P 8100 4850
-F 0 "#PWR08" H 8100 4600 50  0001 C CNN
-F 1 "GND" H 8105 4677 50  0000 C CNN
-F 2 "" H 8100 4850 50  0001 C CNN
-F 3 "" H 8100 4850 50  0001 C CNN
-	1    8100 4850
-	1    0    0    -1
-$EndComp
-$Comp
-L power:VEE #PWR07
-U 1 1 5B8FA652
-P 8100 4650
-F 0 "#PWR07" H 8100 4500 50  0001 C CNN
-F 1 "VEE" H 8117 4823 50  0000 C CNN
-F 2 "" H 8100 4650 50  0001 C CNN
-F 3 "" H 8100 4650 50  0001 C CNN
-	1    8100 4650
-	1    0    0    -1
-$EndComp
-Wire Wire Line
-	7900 4000 8100 4000
-Wire Wire Line
-	8100 4000 8100 3950
-Wire Wire Line
-	7900 4100 8100 4100
-Wire Wire Line
-	8100 4100 8100 4150
-Wire Wire Line
-	7900 4700 8100 4700
-Wire Wire Line
-	8100 4700 8100 4650
-Wire Wire Line
-	7900 4800 8100 4800
-Wire Wire Line
-	8100 4800 8100 4850
-Text GLabel 8000 5300 2    50   Input ~ 0
-VF1
-Text GLabel 8000 5400 2    50   Input ~ 0
-VF2
-Wire Wire Line
-	8000 5300 7900 5300
-Wire Wire Line
-	8000 5400 7900 5400
 Text Notes 4650 1750 0    79   ~ 0
 [-15V;-30V] 0.25A @ 5V in
@@
 L esynr3z_Misc:TestPoint TP3
 U 1 1 5BA30196
-P 5500 4950
-F 0 "TP3" H 5450 5050 50  0000 L CNN
-F 1 "TestPoint" H 5553 4961 50  0001 L CNN
-F 2 "esynr3z_TestPoint:TestPoint_THTPad_D1.5mm_Drill0.7mm" H 5700 4950 50  0001 C CNN
-F 3 "~" H 5700 4950 50  0001 C CNN
-	1    5500 4950
-	1    0    0    -1
+P 5500 5050
+F 0 "TP3" H 5450 5200 50  0000 L CNN
+F 1 "TestPoint" H 5553 5061 50  0001 L CNN
+F 2 "esynr3z_TestPoint:TestPoint_THTPad_D1.5mm_Drill0.7mm" H 5700 5050 50  0001 C CNN
+F 3 "~" H 5700 5050 50  0001 C CNN
+	1    5500 5050
+	-1   0    0    1
 $EndComp
 Wire Wire Line
@@
 Wire Wire Line
 	5500 4000 5500 4050
-Wire Wire Line
-	5500 4950 5500 5000
 Wire Wire Line
 	6100 2100 6100 2150
@@
 Text Notes 4450 3800 0    79   ~ 0
 Filament driver
+$Comp
+L Connector_Generic:Conn_01x04 J1
+U 1 1 5BA3AA64
+P 2950 3400
+F 0 "J1" H 2870 2975 50  0000 C CNN
+F 1 "Conn_01x04" H 2870 3066 50  0000 C CNN
+F 2 "esynr3z_Connector:PinHeader_1x04_P2.54mm_Vertical" H 2950 3400 50  0001 C CNN
+F 3 "~" H 2950 3400 50  0001 C CNN
+	1    2950 3400
+	-1   0    0    1
+$EndComp
+$Comp
+L Connector_Generic:Conn_01x04 J2
+U 1 1 5BA3ACB7
+P 7650 4150
+F 0 "J2" H 7570 3725 50  0000 C CNN
+F 1 "Conn_01x04" H 7570 3816 50  0000 C CNN
+F 2 "esynr3z_Connector:PinHeader_1x04_P2.54mm_Vertical" H 7650 4150 50  0001 C CNN
+F 3 "~" H 7650 4150 50  0001 C CNN
+	1    7650 4150
+	-1   0    0    1
+$EndComp
+$Comp
+L Connector_Generic:Conn_01x04 J3
+U 1 1 5BA40438
+P 7650 4900
+F 0 "J3" H 7570 4475 50  0000 C CNN
+F 1 "Conn_01x04" H 7570 4566 50  0000 C CNN
+F 2 "esynr3z_Connector:PinHeader_1x04_P2.54mm_Vertical" H 7650 4900 50  0001 C CNN
+F 3 "~" H 7650 4900 50  0001 C CNN
+	1    7650 4900
+	-1   0    0    1
+$EndComp
+Text GLabel 7950 4800 2    50   Input ~ 0
+VF1
+Text GLabel 7950 4900 2    50   Input ~ 0
+VF2
+Wire Wire Line
+	7950 4800 7900 4800
+Wire Wire Line
+	7950 4900 7900 4900
+$Comp
+L power:GND #PWR08
+U 1 1 5BA4B596
+P 8050 4300
+F 0 "#PWR08" H 8050 4050 50  0001 C CNN
+F 1 "GND" H 8055 4127 50  0000 C CNN
+F 2 "" H 8050 4300 50  0001 C CNN
+F 3 "" H 8050 4300 50  0001 C CNN
+	1    8050 4300
+	1    0    0    -1
+$EndComp
+$Comp
+L power:VEE #PWR07
+U 1 1 5BA4B59C
+P 8050 3900
+F 0 "#PWR07" H 8050 3750 50  0001 C CNN
+F 1 "VEE" H 8067 4073 50  0000 C CNN
+F 2 "" H 8050 3900 50  0001 C CNN
+F 3 "" H 8050 3900 50  0001 C CNN
+	1    8050 3900
+	1    0    0    -1
+$EndComp
+Wire Wire Line
+	7850 4050 8050 4050
+Wire Wire Line
+	8050 4050 8050 3950
+Wire Wire Line
+	7850 4150 8050 4150
+Wire Wire Line
+	8050 4150 8050 4250
+$Comp
+L power:+5V #PWR05
+U 1 1 5BA512C2
+P 3350 3150
+F 0 "#PWR05" H 3350 3000 50  0001 C CNN
+F 1 "+5V" H 3365 3323 50  0000 C CNN
+F 2 "" H 3350 3150 50  0001 C CNN
+F 3 "" H 3350 3150 50  0001 C CNN
+	1    3350 3150
+	1    0    0    -1
+$EndComp
+$Comp
+L power:GND #PWR06
+U 1 1 5BA512C8
+P 3350 3550
+F 0 "#PWR06" H 3350 3300 50  0001 C CNN
+F 1 "GND" H 3355 3377 50  0000 C CNN
+F 2 "" H 3350 3550 50  0001 C CNN
+F 3 "" H 3350 3550 50  0001 C CNN
+	1    3350 3550
+	1    0    0    -1
+$EndComp
+Wire Wire Line
+	3150 3300 3350 3300
+Wire Wire Line
+	3350 3300 3350 3200
+Wire Wire Line
+	3150 3400 3350 3400
+Wire Wire Line
+	3350 3400 3350 3500
+Wire Wire Line
+	3150 3200 3350 3200
+Connection ~ 3350 3200
+Wire Wire Line
+	3350 3200 3350 3150
+Wire Wire Line
+	3150 3500 3350 3500
+Connection ~ 3350 3500
+Wire Wire Line
+	3350 3500 3350 3550
+Wire Wire Line
+	7850 3950 8050 3950
+Connection ~ 8050 3950
+Wire Wire Line
+	8050 3950 8050 3900
+Wire Wire Line
+	7850 4250 8050 4250
+Connection ~ 8050 4250
+Wire Wire Line
+	8050 4250 8050 4300
+Wire Wire Line
+	7850 4700 7900 4700
+Wire Wire Line
+	7900 4700 7900 4800
+Connection ~ 7900 4800
+Wire Wire Line
+	7900 4800 7850 4800
+Wire Wire Line
+	7850 5000 7900 5000
+Wire Wire Line
+	7900 5000 7900 4900
+Connection ~ 7900 4900
+Wire Wire Line
+	7900 4900 7850 4900
+$Comp
+L esynr3z_Misc:TestPoint TP4
+U 1 1 5BACC723
+P 5950 4000
+F 0 "TP4" H 5900 4100 50  0000 L CNN
+F 1 "TestPoint" H 6003 4011 50  0001 L CNN
+F 2 "esynr3z_TestPoint:TestPoint_THTPad_D1.5mm_Drill0.7mm" H 6150 4000 50  0001 C CNN
+F 3 "~" H 6150 4000 50  0001 C CNN
+	1    5950 4000
+	1    0    0    -1
+$EndComp
+Wire Wire Line
+	5950 4000 5950 4050
+$Comp
+L esynr3z_Misc:TestPoint TP5
+U 1 1 5BAD95CE
+P 5950 5050
+F 0 "TP5" H 5900 5200 50  0000 L CNN
+F 1 "TestPoint" H 6003 5061 50  0001 L CNN
+F 2 "esynr3z_TestPoint:TestPoint_THTPad_D1.5mm_Drill0.7mm" H 6150 5050 50  0001 C CNN
+F 3 "~" H 6150 5050 50  0001 C CNN
+	1    5950 5050
+	-1   0    0    1
+$EndComp
+Wire Wire Line
+	5950 5050 5950 5000
+Wire Wire Line
+	5500 5000 5500 5050
 $EndSCHEMATC

Commit message: Trace all pcb nets
Parts:
- added TP6: TestPoint, esynr3z_TestPoint:TestPoint_THTPad_D1.5mm_Drill0.7mm, symbol esynr3z_Misc:TestPoint
Connections:
- wire segments 163 -> 165
Changed lines of the file:
@@
 EESchema Schematic File Version 4
-LIBS:vfd-ps-cache
 EELAYER 26 0
 EELAYER END
@@
 Wire Wire Line
 	5500 5000 5500 5050
+$Comp
+L esynr3z_Misc:TestPoint TP6
+U 1 1 5BA45EBE
+P 3500 3450
+F 0 "TP6" H 3450 3550 50  0000 L CNN
+F 1 "TestPoint" H 3553 3461 50  0001 L CNN
+F 2 "esynr3z_TestPoint:TestPoint_THTPad_D1.5mm_Drill0.7mm" H 3700 3450 50  0001 C CNN
+F 3 "~" H 3700 3450 50  0001 C CNN
+	1    3500 3450
+	1    0    0    -1
+$EndComp
+Wire Wire Line
+	3500 3450 3500 3500
+Wire Wire Line
+	3500 3500 3350 3500
 $EndSCHEMATC

Commit message: Make project portable
Parts:
- C1, C12, C2, C3, C6, C7, C8: footprint esynr3z_Capacitor:C_1210 -> lib_fp:C_1210; symbol Device:C -> vfd-ps:Device_C
- C10, C14, C5, C9: footprint esynr3z_Capacitor:C_0805 -> lib_fp:C_0805; symbol Device:C -> vfd-ps:Device_C
- C11, C13: footprint esynr3z_Capacitor:CP_Elec_6.3x7.7 -> lib_fp:CP_Elec_6.3x7.7; symbol Device:CP -> vfd-ps:Device_CP
- C15, C4: footprint esynr3z_Capacitor:C_1206 -> lib_fp:C_1206; symbol Device:C -> vfd-ps:Device_C
- D1: footprint esynr3z_Diode:SMA -> lib_fp:SMA; symbol esynr3z_DiodeSchottky:MBRA340 -> vfd-ps:esynr3z_DiodeSchottky_MBRA340
- D2: footprint esynr3z_SOT:SOT-23 -> lib_fp:SOT-23; symbol esynr3z_DiodeZener:BZX84C4V7 -> vfd-ps:esynr3z_DiodeZener_BZX84C4V7
- J1, J2, J3: footprint esynr3z_Connector:PinHeader_1x04_P2.54mm_Vertical -> lib_fp:PinHeader_1x04_P2.54mm_Vertical; symbol Connector_Generic:Conn_01x04 -> vfd-ps:Connector_Generic_Conn_01x04
- JP1: footprint esynr3z_Jumper:SolderJumper-2_P1.3mm_Bridged2Bar_RoundedPad1.0x1.5mm -> lib_fp:SolderJumper-2_P1.3mm_Bridged2Bar_RoundedPad1.0x1.5mm; symbol esynr3z_Misc:SolderJumper_2_Bridged -> vfd-ps:esynr3z_Misc_SolderJumper_2_Bridged
- L1: footprint esynr3z_Inductor:Sumida_CDRH127 -> lib_fp:Sumida_CDRH127; symbol Device:L_Core_Iron -> vfd-ps:Device_L_Core_Iron
- R1, R10, R11, R12, R2, R3, R4, R5, R6, R7, R8, R9: footprint esynr3z_Resistor:R_0805 -> lib_fp:R_0805; symbol Device:R -> vfd-ps:Device_R
- RV1, RV2, RV3: footprint esynr3z_Potentiometer:Bourns_3362P -> lib_fp:Bourns_3362P; symbol Device:R_POT_TRIM -> vfd-ps:Device_R_POT_TRIM
- TP1, TP2, TP3, TP4, TP5, TP6: footprint esynr3z_TestPoint:TestPoint_THTPad_D1.5mm_Drill0.7mm -> lib_fp:TestPoint_THTPad_D1.5mm_Drill0.7mm; symbol esynr3z_Misc:TestPoint -> vfd-ps:esynr3z_Misc_TestPoint
- U1: footprint esynr3z_SO:TI_SO-PowerPAD-8_ThermalVias -> lib_fp:TI_SO-PowerPAD-8_ThermalVias; symbol esynr3z_RegulatorSwitching:TPS54360DDA -> vfd-ps:esynr3z_RegulatorSwitching_TPS54360DDA
- U2: footprint esynr3z_SO:VSSOP-8_3.0x3.0mm_P0.65mm -> lib_fp:VSSOP-8_3.0x3.0mm_P0.65mm; symbol esynr3z_AmplifierAudio:LM4871 -> vfd-ps:esynr3z_AmplifierAudio_LM4871
