File: vfd-ps.sch (KiCad schematic (older format))
At the start: 45 parts, among them J1 Conn_01x04, J2 Conn_01x04, J3 Conn_01x04, U1 TPS54360DDA, U2 LM4871

Commit message: Remove all local libs and switch to submodule library
Parts:
- C1, C12, C2, C3, C6, C7, C8: footprint lib_fp:C_1210 -> esynr3z_Capacitor:C_1210; symbol vfd-ps:Device_C -> esynr3z_Symbol:C
- C10, C14, C5, C9: footprint lib_fp:C_0805 -> esynr3z_Capacitor:C_0805; symbol vfd-ps:Device_C -> esynr3z_Symbol:C
- C11, C13: footprint lib_fp:CP_Elec_6.3x7.7 -> esynr3z_Capacitor:CP_Elec_6.3x7.7; symbol vfd-ps:Device_CP -> esynr3z_Symbol:C_Polar
- C15, C4: footprint lib_fp:C_1206 -> esynr3z_Capacitor:C_1206; symbol vfd-ps:Device_C -> esynr3z_Symbol:C
- D1: footprint lib_fp:SMA -> esynr3z_Diode:SMA; symbol vfd-ps:esynr3z_DiodeSchottky_MBRA340 -> esynr3z_DiodeSchottky:MBRA340
- D2: footprint lib_fp:SOT-23 -> esynr3z_SOT:SOT-23; symbol vfd-ps:esynr3z_DiodeZener_BZX84C4V7 -> esynr3z_DiodeZener:BZX84C4V7
- J1, J2, J3: footprint lib_fp:PinHeader_1x04_P2.54mm_Vertical -> esynr3z_Connector:PinHeader_1x04_P2.54mm_Vertical; symbol vfd-ps:Connector_Generic_Conn_01x04 -> Connector_Generic:Conn_01x04
- JP1: footprint lib_fp:SolderJumper-2_P1.3mm_Bridged2Bar_RoundedPad1.0x1.5mm -> esynr3z_Jumper:SolderJumper-2_P1.3mm_Bridged2Bar_RoundedPad1.0x1.5mm; symbol vfd-ps:esynr3z_Misc_SolderJumper_2_Bridged -> esynr3z_Misc:SolderJumper_2_Bridged
- L1: footprint lib_fp:Sumida_CDRH127 -> esynr3z_Inductor:Sumida_CDRH127; symbol vfd-ps:Device_L_Core_Iron -> esynr3z_Symbol:L_Core_Iron
- R1, R10, R11, R12, R2, R3, R4, R5, R6, R7, R8, R9: footprint lib_fp:R_0805 -> esynr3z_Resistor:R_0805; symbol vfd-ps:Device_R -> esynr3z_Symbol:R
- RV1, RV2, RV3: footprint lib_fp:Bourns_3362P -> esynr3z_Potentiometer:Bourns_3362P; symbol vfd-ps:Device_R_POT_TRIM -> esynr3z_Symbol:R_POT_TRIM
- TP1, TP2, TP3, TP4, TP5, TP6: footprint lib_fp:TestPoint_THTPad_D1.5mm_Drill0.7mm -> esynr3z_TestPoint:TestPoint_THTPad_D1.5mm_Drill0.7mm; symbol vfd-ps:esynr3z_Misc_TestPoint -> esynr3z_Misc:TestPoint
- U1: footprint lib_fp:TI_SO-PowerPAD-8_ThermalVias -> esynr3z_SO:TI_SO-PowerPAD-8_ThermalVias; symbol vfd-ps:esynr3z_RegulatorSwitching_TPS54360DDA -> esynr3z_RegulatorSwitching:TPS54360DDA
- U2: footprint lib_fp:VSSOP-8_3.0x3.0mm_P0.65mm -> esynr3z_SO:VSSOP-8_3.0x3.0mm_P0.65mm; symbol vfd-ps:esynr3z_AmplifierAudio_LM4871 -> esynr3z_AmplifierAudio:LM4871

Commit message: Replace lm4871 footprint
Parts:
- R2: value 16k -> 36k
- R6: value 1k -> 2.2k
- RV1: value 20k -> 50k
Changed lines of the file:
@@
 P 6950 2350
 F 0 "RV1" H 6800 2400 50  0000 C CNN
-F 1 "20k" H 6800 2300 50  0000 C CNN
+F 1 "50k" H 6800 2300 50  0000 C CNN
 F 2 "esynr3z_Potentiometer:Bourns_3362P" H 6950 2350 50  0001 C CNN
 F 3 "~" H 6950 2350 50  0001 C CNN
@@
 P 6950 2750
 F 0 "R2" H 7020 2796 50  0000 L CNN
-F 1 "16k" H 7020 2705 50  0000 L CNN
+F 1 "36k" H 7020 2705 50  0000 L CNN
 F 2 "esynr3z_Resistor:R_0805" V 6880 2750 50  0001 C CNN
 F 3 "~" H 6950 2750 50  0001 C CNN
@@
 P 6950 3150
 F 0 "R6" H 7020 3196 50  0000 L CNN
-F 1 "1k" H 7020 3105 50  0000 L CNN
+F 1 "2.2k" H 7020 3105 50  0000 L CNN
 F 2 "esynr3z_Resistor:R_0805" V 6880 3150 50  0001 C CNN
 F 3 "~" H 6950 3150 50  0001 C CNN

Commit message: Align labels on silk and fab layers
Parts:
- U2: footprint esynr3z_SO:VSSOP-8_3.0x3.0mm_P0.65mm -> esynr3z_SO:SOIC-8_3.9x4.9mm_P1.27mm
Changed lines of the file:
@@
 Title "VFD power supply and filament driver"
 Date ""
-Rev "A"
+Rev "B"
 Comp ""
 Comment1 ""
@@
 F 0 "U2" H 4800 5450 50  0000 C CNN
 F 1 "LM4871" H 5250 5450 50  0000 C CNN
-F 2 "esynr3z_SO:VSSOP-8_3.0x3.0mm_P0.65mm" H 6000 5600 50  0001 C CIN
+F 2 "esynr3z_SO:SOIC-8_3.9x4.9mm_P1.27mm" H 6000 5600 50  0001 C CIN
 F 3 "http://www.ti.com/lit/ds/symlink/lm4871.pdf" H 6050 5700 50  0001 C CNN
 	1    5050 5000
